File: MooresESP32.kicad_sch (KiCad schematic)
At the start: 20 parts, among them J1 PWR, J3 Conn_01x03, J8 Programmer, Q1 BSS138, SW1 SW_Push, SW2 SW_Push, SW3 SW_Push, U1 MCP1700, U4 ESP32-S2-WROVER

Commit message: Updating to KiCAD 8
Parts:
- H1, H2, H3, H4: footprint MountingHole:MountingHole_3mm -> MountingHole:MountingHole_5.5mm
Changed lines of the file:
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@@
 (kicad_sch
-	(version 20231120)
+	(version 20250114)
 	(generator "eeschema")
-	(generator_version "8.0")
+	(generator_version "9.0")
 	(paper "A4")
 	(junction
@@
 			)
 		)
-		(property "Footprint" "MountingHole:MountingHole_3mm"
+		(property "Footprint" "MountingHole:MountingHole_5.5mm"
 			(at 267.97 127 0)
 			(effects
@@
 			)
 		)
-		(property "Footprint" "MountingHole:MountingHole_3mm"
+		(property "Footprint" "MountingHole:MountingHole_5.5mm"
 			(at 247.65 127 0)
 			(effects
@@
 			)
 		)
-		(property "Footprint" "MountingHole:MountingHole_3mm"
+		(property "Footprint" "MountingHole:MountingHole_5.5mm"
 			(at 247.65 139.7 0)
 			(effects
@@
 			)
 		)
-		(property "Footprint" "MountingHole:MountingHole_3mm"
+		(property "Footprint" "MountingHole:MountingHole_5.5mm"
 			(at 267.97 139.7 0)
 			(effects
@@
 		)
 	)
+	(embedded_fonts no)
 )
